File: ChariotFC.kicad_pcb (KiCad board)
At the start: 2 copper layers, 134 parts, among them Q1 2N7002, Q2 BSS138, SW1 1TS009A-1800-5000, SW2 1TS009A-1800-5000, U1 FM25V20A-DGTR_C2952834, U10 SAM-M10Q-00B, U11 INA240A1QDRQ1, U12 TPS62933DRLR, U13 53.6k, U14 B6B-XH-A(LF)(SN)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

Commit message: Joind PDB Batt+ and Batt- pads to LiPo battery input net
Parts:
- moved C1 423.6 mm to (188.6, -373.9)
- moved C10 423.6 mm to (191.5, -373.9)
- moved C11 423.6 mm to (134.1, -329.2)
- moved C12 423.6 mm to (130.6, -328.7)
- moved C13 423.6 mm to (127.6, -328.2)
- moved C14 423.6 mm to (124.7, -328.2)
- moved C15 423.6 mm to (141.2, -329.7)
- moved C16 423.6 mm to (191.5, -363.2)
- moved C17 423.6 mm to (191.5, -361.0)
- moved C18 423.6 mm to (194.4, -373.9)
- moved C19 423.6 mm to (194.4, -371.8)
- moved C2 423.6 mm to (188.6, -371.8)
- moved C20 423.6 mm to (194.4, -369.6)
- moved C21 423.6 mm to (220.0, -374.9)
- moved C22 423.6 mm to (-29.1, -343.9)
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Connections:
- TP21 pad 1: unconnected-(TP21-Pad1) -> CURR_IN
- TP22 pad 1: unconnected-(TP22-Pad1) -> GND
- TP23 pad 1: unconnected-(TP23-Pad1) -> CURR_IN
- TP24 pad 1: unconnected-(TP24-Pad1) -> GND
- TP25 pad 1: unconnected-(TP25-Pad1) -> CURR_IN
- TP26 pad 1: unconnected-(TP26-Pad1) -> GND
- TP27 pad 1: unconnected-(TP27-Pad1) -> CURR_IN
- TP28 pad 1: unconnected-(TP28-Pad1) -> GND
